Commit message: New and exciting stuff

File: robotsim/src/arm_sim/description/urdf/arm.urdf (robot description, URDF)
Before this commit: robot printerArm, 6 links, 5 joints
Links:
- link base_link: mass None -> 10.985
- link link1: mass None -> 5
- link link2: mass None -> 5; geometry visual cylinder length=0.6 radius=0.025
- link link3: mass None -> 5
- link link4: mass None -> 5; geometry visual cylinder length=0.2 radius=0.025
